Commit message: modified youbot urdf

File: urdf/youbot.urdf (robot description, URDF)
Before this commit: robot youbot, 21 links, 20 joints
Links:
- link arm_link_0: mass 0.845 -> 0.961; geometry collision mesh filename=package://youbot_description/meshes/youbot_arm/arm0_convex.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; visual mesh filename=package://youbot_description/meshes/youbot_arm/arm0.dae
- link arm_link_1: mass 2.412 -> 1.39; geometry collision mesh filename=package://youbot_description/meshes/youbot_arm/arm1_convex.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; visual mesh filename=package://youbot_description/meshes/youbot_arm/arm1.dae
- link arm_link_2: mass 1.155 -> 1.318; geometry collision mesh filename=package://youbot_description/meshes/youbot_arm/arm2_convex.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; visual mesh filename=package://youbot_description/meshes/youbot_arm/arm2.dae
- link arm_link_3: mass 0.934 -> 0.821; geometry collision mesh filename=package://youbot_description/meshes/youbot_arm/arm3_convex.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; visual mesh filename=package://youbot_description/meshes/youbot_arm/arm3.dae
- link arm_link_4: mass 0.877 -> 0.769; geometry collision mesh filename=package://youbot_description/meshes/youbot_arm/arm4_convex.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; visual mesh filename=package://youbot_description/meshes/youbot_arm/arm4.dae
- link arm_link_5: mass 0.251 -> 0.687; geometry collision mesh filename=package://youbot_description/meshes/youbot_arm/arm5_convex.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; visual mesh filename=package://youbot_description/meshes/youbot_arm/arm5.dae
- link base_footprint: mass 0.0001 -> 0.1
- link base_laser_front_link: geometry collision mesh filename=package://youbot_description/meshes/sensors/hokuyo_convex.d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; visual mesh filename=package://youbot_description/meshes/sensors/hokuyo.dae
- link base_link: geometry collision mesh filename=package://youbot_description/meshes/youbot_base/base_convex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; visual mesh filename=package://youbot_description/meshes/youbot_base/base.dae
- link gripper_finger_link_l: geometry collision mesh filename=package://youbot_description/meshes/youbot_gripper/finger_c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; visual mesh filename=package://youbot_description/meshes/youbot_gripper/finger.d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
- link gripper_finger_link_r: geometry collision mesh filename=package://youbot_description/meshes/youbot_gripper/finger_c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; visual mesh filename=package://youbot_description/meshes/youbot_gripper/finger.d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
- link gripper_palm_link: geometry collision mesh filename=package://youbot_description/meshes/youbot_gripper/palm_con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; visual mesh filename=package://youbot_description/meshes/youbot_gripper/palm.dae
- link plate_link: mass 1 -> 2.397; geometry collision mesh filename=package://youbot_description/meshes/youbot_plate/plate_conv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; visual mesh filename=package://youbot_description/meshes/youbot_plate/plate.dae
- link wheel_link_bl: mass 0.4 -> 1.4; geometry collision cylinder length=0.0475 radius=0.0475; visual sphere radius=0.0475
- link wheel_link_br: mass 0.4 -> 1.4; geometry collision cylinder length=0.0475 radius=0.0475; visual sphere radius=0.0475
- link wheel_link_fl: mass 0.4 -> 1.4; geometry collision cylinder length=0.0475 radius=0.0475; visual sphere radius=0.0475
- link wheel_link_fr: mass 0.4 -> 1.4; geometry collision cylinder length=0.0475 radius=0.0475; visual sphere radius=0.0475
Joints:
- joint arm_joint_1: limit lower=0 upper=5.89920788889 effort=10000.0 velocity=1.570795 -> lower=0 upper=5.89921287174 effort=9.5 velocity=1.57079632679; origin xyz=0.024 0 0.115 rpy=0 0 2.96705722222 -> xyz=0.024 0 0.096 rpy=0 0 2.96705972839
- joint arm_joint_2: limit lower=0 upper=2.70525805556 effort=10000.0 velocity=1.570795 -> lower=0 upper=2.70526034059 effort=9.5 velocity=1.57079632679; origin xyz=0.033 0 0 rpy=0 -1.13446305556 0 -> xyz=0.033 0 0.019 rpy=0 -1.1344640138 0
- joint arm_joint_3: limit lower=-5.1836235 upper=0 effort=10000.0 velocity=1.570795 -> lower=-5.18362787842 upper=0 effort=6.0 velocity=1.57079632679; origin xyz=0.000 0.000 0.155 rpy=0 2.54817855556 0 -> xyz=0.000 0.000 0.155 rpy=0 2.54818070791 0
- joint arm_joint_4: limit lower=0 upper=3.57792194444 effort=10000.0 velocity=1.570795 -> lower=0 upper=3.57792496659 effort=2.0 velocity=1.57079632679; origin xyz=0.000 0.000 0.135 rpy=0 -1.78896097222 0 -> xyz=0.000 0.000 0.135 rpy=0 -1.78896248329 0
- joint arm_joint_5: limit lower=0 upper=5.84684805556 effort=10000.0 velocity=1.570795 -> lower=0 upper=5.84685299418 effort=1.0 velocity=1.57079632679; origin xyz=0 0 0.114 rpy=0 0 2.92342402778 -> xyz=-0.002 0 0.130 rpy=0 0 2.92342649709
- joint base_laser_front_hokuyo_urg04_laser_joint: origin xyz=0.3 0 -0.03 rpy=3.15 3.15 0 -> xyz=0.3 0 -0.03 rpy=0 0 0
- joint caster_joint_bl: limit (none) -> effort=30 velocity=10; type fixed -> continuous
- joint caster_joint_br: limit (none) -> effort=30 velocity=10; type fixed -> continuous
- joint caster_joint_fl: limit (none) -> effort=30 velocity=10; type fixed -> continuous
- joint caster_joint_fr: limit (none) -> effort=30 velocity=10; type fixed -> continuous
- joint gripper_finger_joint_l: origin xyz=0.046 0.010 0.003  rpy=0 -1.570795 3.14159 -> xyz=0.004 0.008 0.046 rpy=0 0 3.14159265359
- joint gripper_finger_joint_r: origin xyz=0.046 -0.010 0.003 rpy=0 1.570795 0 -> xyz=0.004 -0.008 0.046 rpy=0 0 0
- joint gripper_palm_joint: origin xyz=-0.0027 0 .016 rpy=0 -1.570795 3.14159 -> xyz=0 0 0 rpy=0 0 0
- joint plate_joint: origin xyz=-0.159 0 0.055 rpy=0 0 0 -> xyz=-0.159 0 0.046 rpy=0 0 0
