Commit message: Removed Joint Limits

File: urdf/ur5_robot.urdf (robot description, URDF)
Before this commit: robot ur5, 11 links, 10 joints
Joints:
- joint elbow_joint: limit lower=-6.2831853 upper=6.2831853 effort=150.0 velocity=3.15 -> (none); type revolute -> continuous
- joint shoulder_lift_joint: limit lower=-6.2831853 upper=6.2831853 effort=150.0 velocity=3.15 -> (none); type revolute -> continuous
- joint shoulder_pan_joint: axis 0 0 1 -> (none); limit lower=-6.2831853 upper=6.2831853 effort=150.0 velocity=3.15 -> (none); type revolute -> continuous
- joint wrist_1_joint: limit lower=-6.2831853 upper=6.2831853 effort=28.0 velocity=3.2 -> (none); type revolute -> continuous
- joint wrist_2_joint: limit lower=-6.2831853 upper=6.2831853 effort=28.0 velocity=3.2 -> (none); type revolute -> continuous
- joint wrist_3_joint: limit lower=-6.2831853 upper=6.2831853 effort=28.0 velocity=3.2 -> (none); type revolute -> continuous

File: urdf/wam7.urdf (robot description, URDF)
Before this commit: robot wam, 10 links, 9 joints
Links:
- added link base
Joints:
- added joint shoulder_fixed_joint: type fixed, parent base_link, child base, origin xyz=0.0 0.0 0.346 rpy=0 0 0
- joint base_yaw_joint: limit lower=-2.6 upper=2.6 effort=60 velocity=2.0 -> (none); origin xyz=0 0 0.346 rpy=0 0 0 -> xyz=0 0 0 rpy=0 0 0; parent base_link -> base; type revolute -> continuous
- joint elbow_pitch_joint: limit lower=-0.9 upper=3.14159265359 effort=30 velocity=2.00 -> (none); type revolute -> continuous
- joint palm_yaw_joint: limit lower=-3.0 upper=3.0 effort=10 velocity=2.00 -> (none); type revolute -> continuous
- joint shoulder_pitch_joint: limit lower=-1.985 upper=1.985 effort=60 velocity=2.0 -> (none); type revolute -> continuous
- joint shoulder_yaw_joint: limit lower=-2.8 upper=2.8 effort=45 velocity=2.0 -> (none); type revolute -> continuous
- joint wrist_pitch_joint: limit lower=-1.5707 upper=1.5707 effort=10 velocity=2.00 -> (none); type revolute -> continuous
- joint wrist_yaw_joint: limit lower=-4.55 upper=1.25 effort=10 velocity=2.0 -> (none); type revolute -> continuous

Commit message: fixed shoulder pan joint rotation axis

File: urdf/ur5_robot.urdf (robot description, URDF)
Before this commit: robot ur5, 11 links, 10 joints
Joints:
- joint shoulder_pan_joint: axis (none) -> 0 0 1

Commit message: added ur5 web launchfile

File: urdf/ur5_robot.urdf (robot description, URDF)
Before this commit: robot ur5, 11 links, 10 joints
Links:
- link base_link: mass None -> 4.0
- link forearm_link: mass None -> 2.275
- link shoulder_link: mass None -> 3.7
- link upper_arm_link: mass None -> 8.393
- link wrist_1_link: mass None -> 1.219
- link wrist_2_link: mass None -> 1.219
- link wrist_3_link: mass None -> 0.1879

Commit message: modified UR5 URDF

File: urdf/ur5_robot.urdf (robot description, URDF)
Before this commit: robot ur5, 11 links, 10 joints
Links:
- removed link base
- removed link ee_link
- link base_link: mass None -> 4.0
- link forearm_link: mass None -> 2.275
- link shoulder_link: mass None -> 3.7
- link upper_arm_link: mass None -> 8.393
- link wrist_1_link: mass None -> 1.219
- link wrist_2_link: mass None -> 1.219
- link wrist_3_link: mass None -> 0.1879
Joints:
- removed joint base_link-base_fixed_joint
- removed joint ee_fixed_joint
